Commit message: urdf test

File: robot2.urdf (robot description, URDF)
Before this commit: robot pointone, 7 links, 6 joints
Joints:
- joint hip2leftthigh: axis 1 0 0 -> 0 1 0; origin xyz=0.14 0.0  0.02  -> xyz=0 0 0
- joint hip2rightthigh: axis 1 0 0 -> 0 1 0; origin xyz=-0.14 0 0.02  -> xyz=0 0 0
- joint leftfemur2leftfoot: axis 1 0 0 -> 0 1 0; origin xyz=-0.005 -0.34 -0.3  -> xyz=0 0 0; type revolute -> fixed
- joint leftthigh2leftfemur: axis 1 0 0 -> 0 1 0; origin xyz=0.0 0.18 -0.3  -> xyz=0 0 0
- joint rightfemur2rightfoot: axis 1 0 0 -> 0 1 0; origin xyz=-0.005 0.55 -0.3  -> xyz=0 0 0; type revolute -> fixed
- joint rightthigh2rightfemur: axis 1 0 0 -> 0 1 0; origin xyz=0.0 0.04 -0.3  -> xyz=0 0 0
