Commit message: intertia matrix

File: robot.urdf (robot description, URDF)
Before this commit: robot pointone, 7 links, 6 joints
Links:
- removed link hip
- removed link leftfemur
- removed link leftfoot
- removed link leftthigh
- removed link rightfemur
- removed link rightfoot
- removed link rightthigh
- added link bit1, mass 0.01; collision mesh filename=bit12.stl; visual mesh filename=bit12.stl
- added link bitb, mass 0.01; collision mesh filename=bitb2.stl; visual mesh filename=bitb2.stl
Joints:
- removed joint hip2leftthigh
- removed joint hip2rightthigh
- removed joint leftfemur2leftfoot
- removed joint leftthigh2leftfemur
- removed joint rightfemur2rightfoot
- removed joint rightthigh2rightfemur
- added joint bit12bitb: type revolute, parent bit1, child bitb, origin xyz=0.0 0.0 0.19999999999999996 , axis 1 0 0
